File: kicad/remote/remote.kicad_pcb (KiCad board)
At the start: 2 copper layers, 57.3 x 26.5 mm, 14 parts, among them Y1 Resonator

Commit message: KiCAD project: final design for remote
Parts:
- B1, B2: footprint lock_project:B3F-1000 -> lock_project:SW_PTS645SK43SMTR92LFS
- BAT1: value Battery_Cell -> CR2032
- Y1: value Resonator -> 8MHz; footprint Crystal:Resonator_SMD-3Pin_7.2x3.0mm -> lock_project:CSTNE8M00G550000R0
- renumbered S1 to B3, Radio1 to RADIO1
Connections:
- B1 pad 1: GND -> unconnected-(B1-Pad1)
- B1 pad 2: unconnected-(B1-Pad2) -> /PD5
- B1 pad 3: /PD5 -> unconnected-(B1-Pad3)
- B1 pad 4: unconnected-(B1-Pad4) -> GND
- B2 pad 1: GND -> unconnected-(B2-Pad1)
- B2 pad 2: unconnected-(B2-Pad2) -> /PD6
- B2 pad 3: /PD6 -> unconnected-(B2-Pad3)
- B2 pad 4: unconnected-(B2-Pad4) -> GND
Routing:
- net GND: track 13.9 -> 23.6 mm
- net /PD6: track 22.0 -> 31.1 mm, vias 2 -> 3
- net /PD5: track 39.1 -> 48.0 mm, vias 2 -> 3
- net Net-(CPU1-XTAL1/PB6): track 14.1 -> 15.0 mm
- net Net-(CPU1-XTAL2/PB7): track 5.02 -> 5.56 mm
Other:
- board text added: "3.3v"

Commit message: Revisted remote board design
Parts:
- added D1: LED, LED_SMD:LED_0603_1608Metric, B.Cu at (197.8, 52.2)
- added R2: 4.7k, Resistor_SMD:R_0603_1608Metric, B.Cu at (194.8, 52.2)
- ANT1: value M620720 -> ~
- BAT1: footprint lock_project:Polycase_BATT-HDR-FB -> lock_project:BAT_BK-912
- C1, C2: footprint Capacitor_SMD:C_0201_0603Metric -> Capacitor_SMD:C_0805_2012Metric
- R1: value 10kOhm -> 10k; footprint Resistor_SMD:R_0201_0603Metric -> Resistor_SMD:R_0603_1608Metric
- moved C1 1.93 mm to (195.8, 57.0)
- moved C4 0.93 mm to (195.6, 61.5)
Connections:
- BAT1 pad 1: +3.3V -> GND
- CPU1 pad 25: unconnected-(CPU1-PC2-Pad25) -> /PC2
- ISP1 pad 2: +3.3V -> unconnected-(ISP1-VCC-Pad2)
- R1 pad 1: /RESET -> +3.3V
- R1 pad 2: +3.3V -> /RESET
Routing:
- net +3.3V: track 128.1 -> 80.7 mm
- net /PC2: track 0.00 -> 9.12 mm
- net GND: track 23.6 -> 28.2 mm, vias 18 -> 40
- net /PD5: track 48.0 -> 50.6 mm
- net /RESET: track 76.2 -> 74.5 mm
- net /MOSI: track 39.4 -> 41.0 mm
- net Net-(D1-A): track 0.00 -> 1.42 mm
- net /PD6: track 31.1 -> 32.4 mm
Other:
- board text added: "LED on PC2"
- board text added: "Remote2025 v1 ATmega328P 8MHz, 3.3V"
- board text removed: "3.3v"
- board text removed: "MISO"
- board text removed: "Remote2025 v1"

Commit message: kicad: Fix resistor value on remote
Parts:
- R2: value 4.7k -> 330 Ohm
Changed lines of the file:
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@@
 			)
 		)
-		(property "Value" "4.7k"
+		(property "Value" "330 Ohm"
 			(at 0 -1.43 0)
 			(layer "B.Fab")
